File: ElectricalDesign/TrinityTrack6000/TrinityTrack6000.kicad_sch (KiCad schematic)
At the start: 0 parts

Commit message: Architecture planning
Parts:
- added C1: 100nF, Capacitor_SMD:C_0603_1608Metric_Pad1.08x0.95mm_HandSolder, symbol Device:C_Small
- added U1: STM32G473CETx, Package_QFP:LQFP-48_7x7mm_P0.5mm, symbol MCU_ST_STM32G4:STM32G473CETx
- added U2: MCP23S17_SO, Package_SO:SOIC-28W_7.5x17.9mm_P1.27mm, symbol Interface_Expansion:MCP23S17_SO
- added U3: NRF24L01, Package_DFN_QFN:QFN-20-1EP_4x4mm_P0.5mm_EP2.5x2.5mm, symbol RF:NRF24L01
- added U4: MQ-6, Sensor:MQ-6, symbol Sensor_Gas:MQ-6
Connections:
- new net: U1.23 (VSS), U1.35 (VSS), U1.47 (VSS)
Other:
- title: (none) -> ControlBoard
